Commit message: nub-EE 7DOF arm booster

File: resources/T1_7_dof_arm_serial.urdf (robot description, URDF)
Before this commit: robot T1, 30 links, 29 joints
Links:
- link AL1: geometry visual mesh filename=T1/meshes/AL1.STL
- link AL2: geometry visual mesh filename=T1/meshes/AL2.STL
- link AL3: geometry visual mesh filename=T1/meshes/AL3.STL
- link AL4: geometry visual mesh filename=T1/meshes/AL4.STL
- link AL5: geometry visual mesh filename=T1/meshes/AL5.STL
- link AL6: geometry visual mesh filename=T1/meshes/AL6.STL
- link AR1: geometry visual mesh filename=T1/meshes/AR1.STL
- link AR2: geometry visual mesh filename=T1/meshes/AR2.STL
- link AR3: geometry visual mesh filename=T1/meshes/AR3.STL
- link AR4: geometry visual mesh filename=T1/meshes/AR4.STL
- link AR5: geometry visual mesh filename=T1/meshes/AR5.STL
- link AR6: geometry visual mesh filename=T1/meshes/AR6.STL
- link Ankle_Cross_Left: geometry visual mesh filename=T1/meshes/Ankle_Cross_Left.STL
- link Ankle_Cross_Right: geometry visual mesh filename=T1/meshes/Ankle_Cross_Right.STL
- link H1: geometry visual mesh filename=T1/meshes/H1.STL
- link H2: geometry collision sphere radius=0.08; visual mesh filename=T1/meshes/H2.STL
- link Hip_Pitch_Left: geometry visual mesh filename=T1/meshes/Hip_Pitch_Left.STL
- link Hip_Pitch_Right: geometry visual mesh filename=T1/meshes/Hip_Pitch_Right.STL
- link Hip_Roll_Left: geometry collision cylinder length=0.16 radius=0.05; visual mesh filename=T1/meshes/Hip_Roll_Left.STL
- link Hip_Roll_Right: geometry collision cylinder length=0.16 radius=0.05; visual mesh filename=T1/meshes/Hip_Roll_Right.STL
- link Hip_Yaw_Left: geometry collision cylinder length=0.08 radius=0.05; visual mesh filename=T1/meshes/Hip_Yaw_Left.STL
- link Hip_Yaw_Right: geometry collision cylinder length=0.08 radius=0.05; visual mesh filename=T1/meshes/Hip_Yaw_Right.STL
- link Shank_Left: geometry collision box size=0.1 0.08 0.1; visual mesh filename=T1/meshes/Shank_Left.STL
- link Shank_Right: geometry collision box size=0.1 0.08 0.1; visual mesh filename=T1/meshes/Shank_Right.STL
- link Trunk: geometry collision box size=0.15 0.2 0.3; visual mesh filename=T1/meshes/Trunk.STL
- link Waist: geometry visual mesh filename=T1/meshes/Waist.STL
- link left_foot_link: geometry collision box size=0.223 0.1 0.03; visual mesh filename=T1/meshes/left_foot_link.STL
- link left_hand_link: geometry visual mesh filename=T1/meshes/AL7.STL
- link right_foot_link: geometry collision box size=0.223 0.1 0.03; visual mesh filename=T1/meshes/right_foot_link.STL
- link right_hand_link: geometry visual mesh filename=T1/meshes/AR7.STL

File: resources/T1_with_hands_5dof/T1_with_hands.urdf (robot description, URDF)
Before this commit: robot t1, 83 links, 82 joints
Links:
- removed link left_hand_base
- removed link right_hand_base
- added link left_hand_link, mass 0.6273500000000001; collision mesh filename=meshes/left_hand/base_link.STL; visual mesh filename=meshes/left_hand/base_link.STL
- added link right_hand_link, mass 0.6273500000000001; collision mesh filename=meshes/right_hand/base_link.STL; visual mesh filename=meshes/right_hand/base_link.STL
Joints:
- joint Left_Elbow_Yaw: child left_hand_base -> left_hand_link
- joint Right_Elbow_Yaw: child right_hand_base -> right_hand_link
- joint left_index_1_joint: parent left_hand_base -> left_hand_link
- joint left_little_1_joint: parent left_hand_base -> left_hand_link
- joint left_middle_1_joint: parent left_hand_base -> left_hand_link
- joint left_palm_force_sensor_joint: parent left_hand_base -> left_hand_link
- joint left_ring_1_joint: parent left_hand_base -> left_hand_link
- joint left_thumb_1_joint: parent left_hand_base -> left_hand_link
- joint right_base_joint: child right_hand_base -> right_hand_link
- joint right_index_1_joint: parent right_hand_base -> right_hand_link
- joint right_little_1_joint: parent right_hand_base -> right_hand_link
- joint right_middle_1_joint: parent right_hand_base -> right_hand_link
- joint right_palm_force_sensor_joint: parent right_hand_base -> right_hand_link
- joint right_ring_1_joint: parent right_hand_base -> right_hand_link
- joint right_thumb_1_joint: parent right_hand_base -> right_hand_link
